Commit message: Migrate multibeam sonar to bathymetric_multibeam_sonar plugin
Rename multibeam_sonar to bathymetric_multibeam_sonar throughout:
- New BathymetricMultibeamSonarSystem Gazebo plugin with simplified config
- New wamv_bathymetric_multibeam_sonar xacro macro
- Updated component_config.yaml, macros.xacro, and wamv.urdf
- Added component_config.xacro and thruster_config.yaml
- Commented out DetachableJoint plugin for testing

Co-Authored-By: Claude Opus 4.6 <noreply@anthropic.com>

File: vrx_project11/urdf/macros.xacro (robot description, xacro)
@@ -7,3 +7,4 @@
   <!-- Include extra sensor macros -->
   <xacro:include filename="$(find vrx_project11)/urdf/components/wamv_multibeam_sonar.xacro" />
+  <xacro:include filename="$(find vrx_project11)/urdf/components/wamv_bathymetric_multibeam_sonar.xacro" />
 </robot>

File: vrx_project11/urdf/wamv.urdf (robot description, URDF)
Before this commit: robot WAM-V, 31 links, 30 joints
Links:
- removed link wamv/multibeam_sonar_link
- removed link wamv/multibeam_sonar_post_arm_link
- removed link wamv/multibeam_sonar_post_link
- added link wamv/bathymetric_multibeam_sonar_link, mass 1; collision box size=0.1 0.2 0.2; visual box size=0.1 0.2 0.2
- added link wamv/bathymetric_multibeam_sonar_post_arm_link, mass 0.1; collision cylinder length=0.065 radius=0.008; visual mesh filename=package://vrx_gazebo/models/sensor_post/mesh/sensor_post_ar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
- added link wamv/bathymetric_multibeam_sonar_post_link, mass 1.39185; collision cylinder length=1.5465 radius=0.0076; visual cylinder length=1.5465 radius=0.0076
Joints:
- removed joint wamv/base_to_multibeam_sonar_post_joint
- removed joint wamv/multibeam_sonar_post_arm_to_multibeam_sonar_joint
- removed joint wamv/multibeam_sonar_post_to_multibeam_sonar_post_arm_joint
- added joint wamv/base_to_bathymetric_multibeam_sonar_post_joint: type fixed, parent wamv/base_link, child wamv/bathymetric_multibeam_sonar_post_link, origin xyz=-0.07 0.0 0.52325 rpy=0 0 0
- added joint wamv/bathymetric_multibeam_sonar_post_arm_to_bathymetric_multibeam_sonar_joint: type fixed, parent wamv/bathymetric_multibeam_sonar_post_arm_link, child wamv/bathymetric_multibeam_sonar_link, origin xyz=0.04 0 0.05 rpy=0.0 1.5707963267948966 0.0
- added joint wamv/bathymetric_multibeam_sonar_post_to_bathymetric_multibeam_sonar_post_arm_joint: type fixed, parent wamv/bathymetric_multibeam_sonar_post_link, child wamv/bathymetric_multibeam_sonar_post_arm_link, origin xyz=0.03 0 -0.8732500000000001 rpy=0 0 0
